File: PCB + Schematic/StratoSoar-MK2.1/StratoSoar-MK2.1.kicad_sch (KiCad schematic)
At the start: 112 parts, among them J1 BME280, J10 parachute, J11 VOUT, J12 VIN, J2 AT_ISP, J3 AT_FTDI, J4 Signal, J5 USB_C_Receptacle_USB2.0, J6 JTAG, J7 Power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

Commit message: Update
Parts:
- C16: value C_Small -> 100nF
