File: PCB + Schematic/StratoSoar-MK2.2/StratoSoar-MK2.2.kicad_pcb (KiCad board)
At the start: 4 copper layers, 42 x 87.9 mm, 110 parts, among them J1 BME280, J10 parachute, J11 VOUT, J12 VIN, J2 AT_ISP, J3 AT_FTDI, J4 Signal, J5 USB_C_Receptacle_USB2.0, J6 JTAG, J7 Power, J8 rudder, J9 elevator, Q1 2N3906, Q2 2N3906, Q3 2N3906, Q4 DMN1019USN-13, Q5 DMN1019USN-13, Q6 DMN1019USN-13, SW1 AT_RESET, SW2 EEPROM, SW3 AAA, SW4 PWR_SW, SW5 RESET, U1 MAX-M10S, U2 MPU-9250, U3 ATmega328P-A, U4 AT24C512C-SSHD-T, U5 ATXK-H11-E-32.768KHZ-E50-T3, U6 ATSAMD21G18A-A, U7 MCP1700x-330xxTT, Y1 8MHz, Y2 32.768kHz

Commit message: Update
Other:
- board text added: "SWD"
- board text removed: "JTAG/SWD"
Changed lines of the file:
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@@
 		)
 	)
-	(gr_text "JTAG/SWD"
-		(at 56.896 89.408 270)
+	(gr_text "SWD"
+		(at 56.896 91.948 270)
 		(layer "F.SilkS")
 		(effects

Commit message: PCB
Parts:
- added G***: LOGO, LOGO, F.Cu at (111.4, 117.1)
- added J2: FTDI, Connector_PinHeader_2.54mm:PinHeader_1x06_P2.54mm_Vertical, F.Cu at (55.2, 60.8)
- added J8: Button, Connector_PinHeader_2.54mm:PinHeader_1x02_P2.54mm_Vertical, F.Cu at (92.1, 103.9)
- added J9: VIN, Connector_PinHeader_2.54mm:PinHeader_1x02_P2.54mm_Vertical, F.Cu at (85.5, 110.7)
- added JP2: Voltmeter, Jumper:SolderJumper-3_P1.3mm_Open_RoundedPad1.0x1.5mm_NumberLabels, F.Cu at (76.1, 53.6)
- added JP7: GND Config, Jumper:SolderJumper-2_P1.3mm_Open_RoundedPad1.0x1.5mm, F.Cu at (81.0, 99.6)
- added JP8: VIN Config, Jumper:SolderJumper-2_P1.3mm_Open_RoundedPad1.0x1.5mm, F.Cu at (86.9, 101.5)
- AE1: value Antenna_Chip -> 1575AT43A0040001E; footprint RF_Antenna:RAINSUN_GPS1003 -> 1575AT43A0040E:ANT_1575AT_JOT-L
- C16: value C_Small -> 100nF
- J10: renamed from J8; value rudder -> Rudder
- J11: renamed from J9; value elevator -> Elevator
- J12: renamed from J10; value parachute -> Parachute
- J13: renamed from J3; value AT_FTDI -> GY-91; footprint Connector_PinHeader_2.54mm:PinHeader_1x05_P2.54mm_Vertical -> Connector_PinHeader_2.54mm:1x08_SMD_Pads; moved to B.Cu
- J14: renamed from J11; footprint Connector_PinHeader_2.54mm:Pads_1x02_P2.54mm -> Connector_PinHeader_2.54mm:1x02_SMD_Pads
- J15: renamed from J12; footprint Connector_PinHeader_2.54mm:Pads_1x02_P2.54mm -> Connector_PinHeader_2.54mm:1x02_SMD_Pads
- J5: value USB_C_Receptacle_USB2.0 -> USB-C
- J6: value JTAG -> SWD
- U5: value ATXK-H11-E-32.768KHZ-E50-T3 -> ATXK-H11-E-32.768
- moved J13 27.8 mm to (81.0, 53.1)
- moved J14 3.30 mm to (70.4, 86.6)
- moved J15 3.18 mm to (70.4, 106.3)
- moved J1 2.16 mm to (55.2, 49.9)
- moved AE1 1.90 mm to (87.2, 32.6)
- moved J7 0.51 mm to (92.1, 99.7)
- renumbered J2 to J3, JP7 to JP10, JP2 to JP3, JP3 to JP4, JP4 to JP5, JP5 to JP6, JP6 to JP9
Connections:
- net Net-(JP4-B) renamed ERR_LED
- net Net-(JP5-B) renamed LED
- net Net-(JP6-B) renamed XIN
- net Net-(JP7-B) renamed XOUT
- AE1 pad 1: GND -> unconnected-(AE1-GND-Pad1)
- C16 pad 2: Net-(J3-Pin_5) -> Net-(J15-Pin_6)
- J13 pad 1: GND -> unconnected-(J3-Pin_1-Pad1)
- J13 pad 3: AT_RX -> GND
- J13 pad 4: AT_TX -> AT_SCL
- J13 pad 5: Net-(J3-Pin_5) -> AT_SDA
- R2 pad 1: +BATT -> Net-(JP8-C)
Routing:
- net BST: track 50.3 -> 135.5 mm, vias 3 -> 5
- net A3: track 23.5 -> 103.6 mm, vias 1 -> 2
- net +5V: track 60.7 -> 109.7 mm
- net AT_MISO: track 38.4 -> 56.3 mm, vias 1 -> 2
- net GND: track 153.7 -> 136.6 mm, vias 94 -> 72
- net AT_SCL: track 121.6 -> 138.3 mm, vias 4 -> 5
- net AT_SDA: track 113.0 -> 126.2 mm, vias 11 -> 14
- net SCL: track 105.1 -> 112.3 mm
- net +3.3V: track 96.7 -> 103.5 mm, vias 20 -> 22
- net SDA: track 111.2 -> 116.9 mm
- net Net-(J3-Pin_5): track 3.44 -> 0.00 mm
- net Net-(J15-Pin_6): track 0.00 -> 3.44 mm
- net Net-(JP8-C): track 0.00 -> 2.99 mm
- net -BATT: track 39.0 -> 41.9 mm
- net Net-(SW2-B): track 25.3 -> 28.0 mm
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Other:
- board size 42 x 87.9 mm -> 42 x 83.9 mm
- board text added: "BST"
- board text added: "GY-91"
- board text added: "JP2 = solder 1 for BST or solder 3 for +BATT reference for voltmeter"
- board text added: "JP3 = solder to enable one cell"
- board text added: "JP4 = solder to enable AT LED"
- board text added: "JP5 = solder to enable ERR LED"
- board text added: "JP6 = solder to enable SAMD LED"
- board text added: "JP9/JP10 = solder to enable SAMD crystal"
- board text added: "Servo Pinout"
- board text removed: "JP2 = solder to enable one cell"
- board text removed: "JP3 = solder to enable AT LED"
- board text removed: "JP4 = solder to enable ERR LED"
- board text removed: "JP5 = solder to enable SAMD LED"
- board text removed: "JP6/JP7 = solder to enable SAMD crystal"
- board text removed: "VOUT"
