File: PCB + Schematic/StratoSoar-MK2.2/StratoSoar-MK2.2.kicad_pcb (KiCad board)
At the start: 4 copper layers, 42 x 83.9 mm, 117 parts, among them J1 BME280, J10 Rudder, J11 Elevator, J12 Parachute, J13 GY-91, J14 VOUT, J15 VIN, J2 FTDI, J3 AT_ISP, J4 Signal, J5 USB-C, J6 SWD, J7 Power, J8 Button, J9 VIN, Q1 2N3906, Q2 2N3906, Q3 2N3906, Q4 DMN1019USN-13, Q5 DMN1019USN-13, Q6 DMN1019USN-13, SW1 AT_RESET, SW2 EEPROM, SW3 AAA, SW4 PWR_SW, SW5 RESET, U1 MAX-M10S, U2 MPU-9250, U3 ATmega328P-A, U4 AT24C512C-SSHD-T, U5 ATXK-H11-E-32.768, U6 ATSAMD21G18A-A, U7 MCP1700x-330xxTT, Y1 8MHz, Y2 32.768kHz

Commit message: PCB
Other:
- board text added: "JP7 = solder to bridge GND to -BATT"
- board text added: "JP8 = solder to bridge BST and +BATT"

Commit message: Finish new PCB
Parts:
- removed the G*** at (111.4, 117.1)
- turned AE1 to 90 degrees
Connections:
- AE1 pad 1: unconnected-(AE1-GND-Pad1) -> RF
- AE1 pad 2: RF -> unconnected-(AE1-GND-Pad2)
Routing:
- net GND: vias 72 -> 73
Other:
- board text added: "FTDI"
- board text added: "NC"

Commit message: PCB, Code
Other:
- board text added: "~ + -"
