File: PCB + Schematic/StratoSoar-MK2.2/StratoSoar-MK2.2.kicad_sch (KiCad schematic)
At the start: 108 parts, among them J1 BME280, J10 parachute, J11 VOUT, J12 VIN, J2 AT_ISP, J3 AT_FTDI, J4 Signal, J5 USB_C_Receptacle_USB2.0, J6 JTAG, J7 Power, J8 rudder, J9 elevator, Q1 2N3906, Q2 2N3906, Q3 2N3906, Q4 DMN1019USN-13, Q5 DMN1019USN-13, Q6 DMN1019USN-13, SW1 AT_RESET, SW2 EEPROM, SW3 AAA, SW4 PWR_SW, SW5 RESET, U1 MAX-M10S, U2 MPU-9250, U3 ATmega328P-A, U4 AT24C512C-SSHD-T, U5 ATXK-H11-E-32.768KHZ-E50-T3, U6 ATSAMD21G18A-A, U7 MCP1700x-330xxTT, Y1 8MHz, Y2 32.768kHz

Commit message: Update
Parts:
- J6: value JTAG -> SWD
Changed lines of the file:
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@@
 		(fields_autoplaced yes)
 		(property "Reference" "J6"
-			(at 189.738 144.78 0)
+			(at 189.23 144.7799 0)
 			(effects
 				(font
@@
 			)
 		)
-		(property "Value" "JTAG"
-			(at 189.738 147.32 0)
+		(property "Value" "SWD"
+			(at 189.23 147.3199 0)
 			(effects
 				(font

Commit message: PCB
Parts:
- removed J3: AT_FTDI, Connector_PinHeader_2.54mm:PinHeader_1x05_P2.54mm_Vertical, symbol Connector_Generic:Conn_01x05
- added J13: GY-91, Connector_PinHeader_2.54mm:1x08_SMD_Pads, symbol Connector_Generic:Conn_01x08
- added J2: FTDI, Connector_PinHeader_2.54mm:PinHeader_1x06_P2.54mm_Vertical, symbol Connector_Generic:Conn_01x06
- added J8: Button, Connector_PinHeader_2.54mm:PinHeader_1x02_P2.54mm_Vertical, symbol Connector_Generic:Conn_01x02
- added J9: VIN, Connector_PinHeader_2.54mm:PinHeader_1x02_P2.54mm_Vertical, symbol Connector_Generic:Conn_01x02
- added JP2: Voltmeter, Jumper:SolderJumper-3_P1.3mm_Open_RoundedPad1.0x1.5mm_NumberLabels, symbol Jumper:SolderJumper_3_Open
- added JP7: GND Config, Jumper:SolderJumper-2_P1.3mm_Open_RoundedPad1.0x1.5mm, symbol Jumper:SolderJumper_2_Open
- added JP8: VIN Config, Jumper:SolderJumper-2_P1.3mm_Open_RoundedPad1.0x1.5mm, symbol Jumper:SolderJumper_2_Open
- AE1: value Antenna_Chip -> 1575AT43A0040001E; footprint RF_Antenna:RAINSUN_GPS1003 -> 1575AT43A0040E:ANT_1575AT_JOT-L
- J10: renamed from J8; value rudder -> Rudder
- J11: renamed from J9; value elevator -> Elevator
- J12: renamed from J10; value parachute -> Parachute
- J14: renamed from J11; footprint Connector_PinHeader_2.54mm:Pads_1x02_P2.54mm -> Connector_PinHeader_2.54mm:1x02_SMD_Pads
- J15: renamed from J12; footprint Connector_PinHeader_2.54mm:Pads_1x02_P2.54mm -> Connector_PinHeader_2.54mm:1x02_SMD_Pads
- J5: value USB_C_Receptacle_USB2.0 -> USB-C
- U5: value ATXK-H11-E-32.768KHZ-E50-T3 -> ATXK-H11-E-32.768
- renumbered J2 to J3, JP7 to JP10, JP2 to JP3, JP3 to JP4, JP4 to JP5, JP5 to JP6, JP6 to JP9
Connections:
- net +3.3V: now also J13.2 (Pin_2)
- net +5V: now also J2.3 (Pin_3)
- net +BATT: now also JP2.3 (B), JP8.1 (A); no longer R2.1
- net -BATT: now also JP7.1 (A)
- net A3: now also J8.1 (Pin_1)
- net AT_RX: now also J2.4 (Pin_4)
- net AT_SCL: now also J13.4 (Pin_4)
- net AT_SDA: now also J13.5 (Pin_5)
- net AT_TX: now also J2.5 (Pin_5)
- net BST: now also J9.2 (Pin_2), JP2.1 (A), JP8.2 (B)
- net GND: now also J13.3 (Pin_3), J2.1 (Pin_1), J8.2 (Pin_2), J9.1 (Pin_1), JP7.2 (B); no longer AE1.1 (GND)
- net at C16.2: now also J2.6 (Pin_6)
- net ERR_LED: now reaches JP5.2 (B), U6.3 (PA02)
- net XIN: now reaches C24.2, JP9.2 (B), U6.1 (PA00)
- net LED: now reaches JP6.2 (B), U6.26 (PA17)
- net XOUT: now reaches JP10.2 (B), U6.2 (PA01)
- new net: JP2.2 (C), R2.1
Other:
- note added: "32.768 kHz TCXO"
- note added: "32.768 kHz XO"
- note added: "8MHz XTAL"
- note added: "ATMega ISP"
- note added: "ATMega328P - Secondary MCU"
- note added: "Battery"
- note added: "Boost converter (5V)"
- note added: "Elevator servo and FET"
- note added: "Extra decoupling capacitors"
- note added: "FTDI"
- note added: "I2C pullup resistors"
- note added: "IMU"
- note added: "Indicator LED"
- note added: "Indicator LEDs"
- note added: "Linear reg"
- note added: "MPU-9250 (IMU)"
- note added: "Mounting holes"
- note added: "Other circuitry and parts"
- note added: "Parachute servo and FET"
- note added: "Power headers"
- note added: "Power jumpers"
- note added: "Reset circuit"
- note added: "Rudder servo and FET"
- note added: "SAMD21G18A - Main MCU"
- note added: "Sensors/peripherals"
- note added: "Signal headers"
- note added: "USB-C (data and power)"
- note removed: "ATMega"
- note removed: "ATMega ISP Programming"
- note removed: "Boost converter (5v)"
- note removed: "Extra Decoupling Capacitors"
- note removed: "Headers"
- note removed: "MPU9250 (Gyro/Accel/Magnetometer)"
- note removed: "Mounting Holes"
- note removed: "Note to self: It may be difficult and expensive to design for an any voltage battery input. The reason I'm thinking this is because it will need another voltage regulator to drop down to 3.3v. Unless the voltage is kept under 5.2v, a boost converter will be needed to power the servos. We don't want to pwoer the servos from a 12v battery. So, the current from the battery will first need to go thro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"
- note removed: "Notes/To-Do: - Change crystal. - Add a diode for reverse boost converter voltage protection. - Add a port for the wireless serial. - Change reference voltage resistors. - Take away pins for the wireless serial. - Intergrate a switch to turn the thing off from code. - Add a ground plane. - mcuDude's MiniCore should be used to burn a bootloader on the ATMega that uses the internal 8 MHz crystal. - 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"
- note removed: "SAMD"
- note removed: "Servo and FETs"
- note removed: "USB-C"
- company: (none) -> New England Wheather Balloon Society
- title: (none) -> StratoSoar MK2.2
- moved on the sheet: AE1, BT1, BT2, C1, C10, C11, C12, C13, C14, C15, C16, C17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

Commit message: Finish new PCB
Connections:
- net RF: now also AE1.1 (FEED); no longer AE1.2 (RF)
Changed lines of the file:
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@@
 			)
 		)
-		(property "Description" ""
+		(property "Description" "Ceramic chip antenna with pin for PCB trace"
 			(at 331.47 382.27 0)
 			(effects
